File: caon-plate/caon-plate.kicad_sch (KiCad schematic)
At the start: 175 parts, among them J1 OLED_128x32, SW45 EC11 ENCODER 1, SW60 EC11 ENCODER 1, U1 SuperMini nRF52840, U2 74HC595, U3 74HC595

Commit message: Plate Update
Parts:
- SW1, SW10, SW11, SW12, SW13, SW14, SW15, SW16, SW17, SW18, SW19, SW2, SW20, SW21, SW22, SW23, SW24, SW25, SW26, SW27, SW28, SW29, SW3, SW30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: footprint Caon_Footprint:SW_PUSH_6mm -> Caon_Footprint:Hotswap_MX_Plated_1u
