File: caon-plate/caon-plate.kicad_pcb (KiCad board)
At the start: 2 copper layers, 304.8 x 95.2 mm, 73 parts

Commit message: Update
Parts:
- added REF**: OLED_128x32, ScottoKeebs_Components:OLED_128x32, F.Cu at (311.1, 47.6)
Other:
- outline, holes or cut-outs redrawn
Changed lines of the file:
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@@
 		(allow_soldermask_bridges_in_footprints no)
 		(tenting front back)
-		(grid_origin 15.875 111.125)
+		(grid_origin 15.875 15.875)
 		(pcbplotparams
 			(layerselection 0x00000000_00000000_55555555_5755f5ff)
@@
 		)
 	)
+	(footprint "ScottoKeebs_Components:OLED_128x32"
+		(layer "F.Cu")
+		(at 311.15 47.625 90)
+		(property "Reference" "REF**"
+			(at 7.75 10 90)
+			(layer "F.SilkS")
+			(hide yes)
+			(effects
+				(font
+					(size 1 1)
+					(thickness 0.15)
+				)
+			)
+		)
+		(property "Value" "OLED_128x32"
+			(at 0 0 90)
+			(layer "F.Fab")
+			(effects
+				(font
+					(size 1 1)
+					(thickness 0.15)
+				)
+			)
+		)
+		(property "Datasheet" ""
+			(at 0 0 90)
+			(layer "F.Fab")
+			(hide yes)
+			(effects
+				(font
+					(size 1.27 1.27)
+					(thickness 0.15)
+				)
+			)
+		)
+		(property "Description" ""
+			(at 0 0 90)
+			(layer "F.Fab")
+			(hide yes)
+			(effects
+				(font
+					(size 1.27 1.27)
+					(thickness 0.15)
+				)
+			)
+		)
+		(attr through_hole exclude_from_pos_files)
+		(fp_line
+			(start 32.25 -5.75)
+			(end 32.25 6.25)
+			(stroke
+				(width 0.12)
+				(type solid)
+			)
+			(layer "Dwgs.User")
+		)
+		(fp_line
+			(start 30 -5.75)
+			(end 30 6.25)
+			(stroke
+				(width 0.12)
+				(type solid)
+			)
+			(layer "Dwgs.User")
+		)
+		(fp_line
+			(start 0 -5.75)
+			(end 0 6.25)
+			(stroke
+				(width 0.12)
+				(type solid)
+			)
+			(layer "Dwgs.User")
+		)
+		(fp_line
+			(start -5.75 -5.75)
+			(end 32.25 -5.75)
+			(stroke
+				(width 0.12)
+				(type solid)
+			)
+			(layer "Dwgs.User")
+		)
+		(fp_line
+			(start -5.75 -5.75)
+			(end -5.75 6.25)
+			(stroke
+				(width 0.12)
+				(type solid)
+			)
+			(layer "Dwgs.User")
+		)
+		(fp_line
+			(start 1.31 -3.53)
+			(end 23.69 -3.53)
+			(stroke
+				(width 0.12)
+				(type solid)
+			)
+			(layer "Dwgs.User")
+		)
+		(fp_line
+			(start 1.31 -3.53)
+			(end 1.31 1.99)
+			(stroke
+				(width 0.12)
+				(type solid)
+			)
+			(layer "Dwgs.User")
+		)
+		(fp_line
+			(start 23.69 1.99)
+			(end 23.69 -3.53)
+			(stroke
+				(width 0.12)
+				(type solid)
+			)
+			(layer "Dwgs.User")
+		)
+		(fp_line
+			(start 1.31 1.99)
+			(end 23.69 1.99)
+			(stroke
+				(width 0.12)
+				(type solid)
+			)
+			(layer "Dwgs.User")
+		)
+		(fp_line
+			(start 32.25 6.25)
+			(end -5.75 6.25)
+			(stroke
+				(width 0.12)
+				(type solid)
+			)
+			(layer "Dwgs.User")
+		)
+		(pad "1" thru_hole rect
+			(at -4.15 4.05 270)
+			(size 1.7 1.7)
+			(drill 1)
+			(layers "*.Cu" "*.Mask")
+			(remove_unused_layers no)
+		)
+		(pad "2" thru_hole oval
+			(at -4.15 1.51 270)
+			(size 1.7 1.7)
+			(drill 1)
+			(layers "*.Cu" "*.Mask")
+			(remove_unused_layers no)
+		)
+		(pad "3" thru_hole oval
+			(at -4.15 -1.03 270)
+			(size 1.7 1.7)
+			(drill 1)
+			(layers "*.Cu" "*.Mask")
+			(remove_unused_layers no)
+		)
+		(pad "4" thru_hole oval
+			(at -4.15 -3.57 270)
+			(size 1.7 1.7)
+			(drill 1)
+			(layers "*.Cu" "*.Mask")
+			(remove_unused_layers no)
+		)
+		(embedded_fonts no)
+		(model "${SCOTTOKEEBS_KICAD}/3dmodels/ScottoKeebs_Components.3dshapes/OLED_128x32.step"
+			(offset
+				(xyz 13.4 -0.254 7)
+			)
+			(scale
+				(xyz 1 1 1)
+			)
+			(rotate
+				(xyz -0 -0 -0)
+			)
+		)
+	)
 	(footprint "ScottoKeebs_Cutout:Cutout_MX_1.00u"
 		(layer "F.Cu")
@@
 		)
 	)
+	(gr_circle
+		(center 311.15 82.55)
+		(end 314.65 82.55)
+		(stroke
+			(width 0.05)
+			(type solid)
+		)
+		(fill no)
+		(layer "Edge.Cuts")
+	)
 	(gr_line
 		(start 320.675 111.125)
@@
 		(layer "Edge.Cuts")
 	)
+	(gr_circle
+		(center 311.15 63.5)
+		(end 314.65 63.5)
+		(stroke
+			(width 0.05)
+			(type solid)
+		)
+		(fill no)
+		(layer "Edge.Cuts")
+	)

Commit message: Schematic update
Parts:
- REF**: footprint Caon_Footprint:SuperMini_NiceNano_USBdn -> Caon_Footprint:SuperMini_NiceNano_platecutout
Changed lines of the file:
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@@
 		)
 	)
-	(footprint "Caon_Footprint:SuperMini_NiceNano_USBdn"
+	(footprint "Caon_Footprint:SuperMini_NiceNano_platecutout"
 		(layer "F.Cu")
 		(at 311.15 34.13125)
@@
 			(unlocked yes)
 			(layer "F.Fab")
+			(hide yes)
 			(effects
 				(font
@@
 			(layer "F.SilkS")
 		)
+		(fp_rect
+			(start -8.628 -17.01)
+			(end -6.628 14.47)
+			(stroke
+				(width 0.05)
+				(type solid)
+			)
+			(fill no)
+			(layer "Edge.Cuts")
+		)
+		(fp_rect
+			(start 6.628 -17.01)
+			(end 8.628 14.47)
+			(stroke
+				(width 0.05)
+				(type solid)
+			)
+			(fill no)
+			(layer "Edge.Cuts")
+		)
 		(fp_text user "024"
 			(at 9.12 3.81 0)
@@
 			)
 		)
-		(pad "1" thru_hole circle
-			(at 7.62 -13.97)
+		(pad "" thru_hole oval
+			(at -0.5334 10.87628 345)
+			(size 1.8 3.8)
+			(drill 1
+				(offset 0 -1)
+			)
+			(layers)
+			(remove_unused_layers no)
+		)
+		(pad "" thru_hole circle
+			(at 0 8.89)
 			(size 1.8 1.8)
 			(drill 1)
-			(layers "*.Cu" "*.Mask")
+			(layers)
 			(remove_unused_layers no)
 		)
-		(pad "2" thru_hole circle
-			(at 7.62 -11.43)
+		(pad "" thru_hole oval
+			(at 2.0066 10.87628 345)
+			(size 1.8 3.8)
+			(drill 1
+				(offset 0 -1)
+			)
+			(property pad_prop_castellated)
+			(layers)
+			(remove_unused_layers no)
+		)
+		(pad "" thru_hole circle
+			(at 2.54 8.89)
 			(size 1.8 1.8)
 			(drill 1)
-			(layers "*.Cu" "*.Mask")
+			(layers)
 			(remove_unused_layers no)
 		)
-		(pad "3" thru_hole roundrect
-			(at 7.62 -8.89)
-			(size 1.8 1.8)
-			(drill 1)
-			(layers "*.Cu" "*.Mask")
-			(remove_unused_layers no)
-			(roundrect_rratio 0.25)
-		)
-		(pad "4" thru_hole roundrect
-			(at 7.62 -6.35)
-			(size 1.8 4.34)
-			(drill 1
-				(offset 0 -1.27)
-			)
-			(layers "*.Cu" "*.Mask")
-			(remove_unused_layers no)
-			(roundrect_rratio 0.25)
-		)
-		(pad "5" thru_hole circle
-			(at 7.62 -3.81)
-			(size 1.8 1.8)
-			(drill 1)
-			(layers "*.Cu" "*.Mask")
-			(remove_unused_layers no)
-		)
-		(pad "6" thru_hole circle
-			(at 7.62 -1.27)
-			(size 1.8 1.8)
-			(drill 1)
-			(layers "*.Cu" "*.Mask")
-			(remove_unused_layers no)
-		)
-		(pad "7" thru_hole circle
-			(at 7.62 1.27)
-			(size 1.8 1.8)
-			(drill 1)
-			(layers "*.Cu" "*.Mask")
-			(remove_unused_layers no)
-		)
-		(pad "8" thru_hole circle
-			(at 7.62 3.81)
-			(size 1.8 1.8)
-			(drill 1)
-			(layers "*.Cu" "*.Mask")
-			(remove_unused_layers no)
-		)
-		(pad "9" thru_hole circle
-			(at 7.62 6.35)
-			(size 1.8 1.8)
-			(drill 1)
-			(layers "*.Cu" "*.Mask")
-			(remove_unused_layers no)
-		)
-		(pad "10" thru_hole circle
-			(at 7.62 8.89)
-			(size 1.8 1.8)
-			(drill 1)
-			(layers "*.Cu" "*.Mask")
-			(remove_unused_layers no)
-		)
-		(pad "11" thru_hole circle
-			(at 7.62 11.43)
-			(size 1.8 1.8)
-			(drill 1)
-			(layers "*.Cu" "*.Mask")
-			(remove_unused_layers no)
-		)
-		(pad "12" thru_hole circle
-			(at 7.62 13.97)
-			(size 1.8 1.8)
-			(drill 1)
-			(layers "*.Cu" "*.Mask")
-			(remove_unused_layers no)
-		)
-		(pad "13" thru_hole oval
-			(at -7.62 -13.97)
-			(size 1.8 4.34)
-			(drill 1
-				(offset 0 -1.27)
-			)
-			(layers "*.Cu" "*.Mask")
-			(remove_unused_layers no)
-		)
-		(pad "14" thru_hole roundrect
-			(at -7.62 -11.43)
-			(size 1.8 1.8)
-			(drill 1)
-			(layers "*.Cu" "*.Mask")
-			(remove_unused_layers no)
-			(roundrect_rratio 0.25)
-		)
-		(pad "15" thru_hole circle
-			(at -7.62 -8.89)
-			(size 1.8 1.8)
-			(drill 1)
-			(layers "*.Cu" "*.Mask")
-			(remove_unused_layers no)
-		)
-		(pad "16" thru_hole circle
-			(at -7.62 -6.35)
-			(size 1.8 1.8)
-			(drill 1)
-			(layers "*.Cu" "*.Mask")
-			(remove_unused_layers no)
-		)
-		(pad "17" thru_hole circle
-			(at -7.62 -3.81)
-			(size 1.8 1.8)
-			(drill 1)
-			(layers "*.Cu" "*.Mask")
-			(remove_unused_layers no)
-		)
-		(pad "18" thru_hole circle
-			(at -7.62 -1.27)
-			(size 1.8 1.8)
-			(drill 1)
-			(layers "*.Cu" "*.Mask")
-			(remove_unused_layers no)
-		)
-		(pad "19" thru_hole circle
-			(at -7.62 1.27)
-			(size 1.8 1.8)
-			(drill 1)
-			(layers "*.Cu" "*.Mask")
-			(remove_unused_layers no)
-		)
-		(pad "20" thru_hole circle
-			(at -7.62 3.81)
-			(size 1.8 1.8)
-			(drill 1)
-			(layers "*.Cu" "*.Mask")
-			(remove_unused_layers no)
-		)
-		(pad "21" thru_hole circle
-			(at -7.62 6.35)
-			(size 1.8 1.8)
-			(drill 1)
-			(layers "*.Cu" "*.Mask")
-			(remove_unused_layers no)
-		)
-		(pad "22" thru_hole circle
-			(at -7.62 8.89)
-			(size 1.8 1.8)
-			(drill 1)
-			(layers "*.Cu" "*.Mask")
-			(remove_unused_layers no)
-		)
-		(pad "23" thru_hole circle
-			(at -7.62 11.43)
-			(size 1.8 1.8)
-			(drill 1)
-			(layers "*.Cu" "*.Mask")
-			(remove_unused_layers no)
-		)
-		(pad "24" thru_hole circle
-			(at -7.62 13.97)
-			(size 1.8 1.8)
-			(drill 1)
-			(layers "*.Cu" "*.Mask")
-			(remove_unused_layers no)
-		)
-		(pad "25" thru_hole oval
+		(pad "" thru_hole oval
 			(at 4.5466 10.87628 345)
 			(size 1.8 3.8)
@@
 				(offset 0 -1)
 			)
-			(layers "*.Cu" "*.Mask")
+			(layers)
 			(remove_unused_layers no)
 		)
-		(pad "25" thru_hole circle
+		(pad "" thru_hole circle
 			(at 5.08 8.89 345)
 			(size 1.8 1.8)
 			(drill 1)
-			(layers "*.Cu" "*.Mask")
+			(layers)
 			(remove_unused_layers no)
 		)
-		(pad "26" thru_hole oval
-			(at 2.0066 10.87628 345)
-			(size 1.8 3.8)
-			(drill 1
-				(offset 0 -1)
-			)
-			(layers "*.Cu" "*.Mask")
-			(remove_unused_layers no)
-		)
-		(pad "26" thru_hole circle
-			(at 2.54 8.89)
-			(size 1.8 1.8)
-			(drill 1)
-			(layers "*.Cu" "*.Mask")
-			(remove_unused_layers no)
-		)
-		(pad "27" thru_hole oval
-			(at -0.5334 10.87628 345)
-			(size 1.8 3.8)
-			(drill 1
-				(offset 0 -1)
-			)
-			(layers "*.Cu" "*.Mask")
-			(remove_unused_layers no)
-		)
-		(pad "27" thru_hole circle
-			(at 0 8.89)
-			(size 1.8 1.8)
-			(drill 1)
-			(layers "*.Cu" "*.Mask")
-			(remove_unused_layers no)
-		)
-		(pad "28" thru_hole roundrect
-			(at 7.62 -16.51)
-			(size 1.8 1.8)
-			(drill 1)
-			(layers "*.Cu" "*.Mask")
-			(remove_unused_layers no)
-			(roundrect_rratio 0.25)
-		)
-		(pad "29" thru_hole circle
-			(at -7.62 -16.51)
-			(size 1.8 1.8)
-			(drill 1)
-			(layers "*.Cu" "*.Mask" "B.Adhes")
-			(remove_unused_layers no)
-		)
 		(embedded_fonts no)
-		(model "E:/PROJECT/Caon65/3d/Nice_Nano_V2_Flipped.step"
+		(model "E:/PROJECT/Personal-Kicad-Library/3d/Nice_Nano_V2_Flipped.step"
 			(offset
 				(xyz -0.1 1.3 3)
@@
 			)
 			(rotate
-				(xyz 0 0 0)
-			)
-		)
+				(xyz -0 -0 -0)
+			)
+		)

Commit message: Plate design v1.0
Parts:
- REF**: footprint ScottoKeebs_Components:OLED_128x32 -> Caon_Footprint:OLED_128x32
- moved REF** 3.17 mm to (311.1, 50.8)

Commit message: Plate Update
Parts:
- added REF**: MountingHole_2.2mm_M2, MountingHole:MountingHole_2.2mm_M2, F.Cu at (311.1, 20.6)
- added REF**: MountingHole_2.2mm_M2, MountingHole:MountingHole_2.2mm_M2, F.Cu at (34.9, 20.6)
- added REF**: MountingHole_2.2mm_M2, MountingHole:MountingHole_2.2mm_M2, F.Cu at (301.6, 106.4)
- added REF**: MountingHole_2.2mm_M2, MountingHole:MountingHole_2.2mm_M2, F.Cu at (46.0, 63.5)
- added REF**: MountingHole_2.2mm_M2, MountingHole:MountingHole_2.2mm_M2, F.Cu at (225.4, 20.6)
- added REF**: MountingHole_2.2mm_M2, MountingHole:MountingHole_2.2mm_M2, F.Cu at (34.9, 106.4)
- added REF**: MountingHole_2.2mm_M2, MountingHole:MountingHole_2.2mm_M2, F.Cu at (111.1, 20.6)
- added REF**: MountingHole_2.2mm_M2, MountingHole:MountingHole_2.2mm_M2, F.Cu at (277.8, 63.5)
- added REF**: MountingHole_2.2mm_M2, MountingHole:MountingHole_2.2mm_M2, F.Cu at (163.5, 63.5)
- added REF**: MountingHole_2.2mm_M2, MountingHole:MountingHole_2.2mm_M2, F.Cu at (94.5, 106.4)
- added REF**: MountingHole_2.2mm_M2, MountingHole:MountingHole_2.2mm_M2, F.Cu at (204.0, 106.4)
- moved REF** 0.06 mm to (106.4, 101.6)
