File: caon-plate/caon-plate.kicad_pcb (KiCad board)
At the start: 2 copper layers, 304.8 x 95.2 mm, 85 parts

Commit message: Plate update
Parts:
- removed the REF** at (106.4, 82.5)
- removed the REF** at (192.1, 63.5)
- removed the REF** at (111.1, 44.5)
- removed the REF** at (134.9, 63.5)
- removed the REF** at (77.8, 63.5)
- removed the REF** at (63.5, 101.6)
- removed the REF** at (96.8, 63.5)
- removed the REF** at (101.6, 25.4)
- removed the REF** at (292.1, 25.4)
- removed the REF** at (177.8, 25.4)
- removed the REF** at (149.2, 44.5)
- removed the REF** at (139.7, 25.4)
- removed the REF** at (244.5, 44.5)
- removed the REF** at (234.9, 101.6)
- removed the REF** at (163.5, 82.5)
- removed the REF** at (168.3, 101.6)
- removed the REF** at (92.1, 44.5)
- removed the REF** at (149.2, 101.6)
- removed the REF** at (196.8, 25.4)
- removed the REF** at (158.8, 25.4)
- removed the REF** at (144.5, 82.5)
- removed the REF** at (182.6, 82.5)
- removed the REF** at (230.2, 63.5)
- removed the REF** at (168.3, 44.5)
- removed the REF** at (58.7, 63.5)
- removed the REF** at (249.2, 63.5)
- removed the REF** at (49.2, 82.5)
- removed the REF** at (263.5, 44.5)
- removed the REF** at (268.3, 63.5)
- removed the REF** at (120.7, 25.4)
- removed the REF** at (234.9, 25.4)
- removed the REF** at (211.1, 63.5)
- removed the REF** at (54.0, 44.5)
- removed the REF** at (273.1, 101.6)
- removed the REF** at (82.5, 101.6)
- removed the REF** at (154.0, 63.5)
- removed the REF** at (292.1, 101.6)
- removed the REF** at (225.4, 44.5)
- removed the REF** at (115.9, 63.5)
- removed the REF** at (201.6, 82.5)
- removed the REF** at (292.1, 82.5)
- removed the REF** at (239.7, 82.5)
- removed the REF** at (215.9, 101.6)
- removed the REF** at (254.0, 25.4)
- removed the REF** at (273.1, 25.4)
- removed the REF** at (44.5, 101.6)
- removed the REF** at (82.5, 25.4)
- removed the REF** at (87.3, 82.5)
- removed the REF** at (220.7, 82.5)
- removed the REF** at (215.9, 25.4)
- removed the REF** at (130.2, 101.6)
- removed the REF** at (173.0, 63.5)
- removed the REF** at (130.2, 44.5)
- removed the REF** at (254.0, 101.6)
- removed the REF** at (25.4, 101.6)
- removed the REF** at (25.4, 25.4)
- removed the REF** at (68.3, 82.5)
- removed the REF** at (44.5, 25.4)
- removed the REF** at (73.0, 44.5)
- removed the REF** at (311.1, 101.6)
- removed the REF** at (187.3, 44.5)
- removed the REF** at (206.4, 44.5)
- removed the REF** at (125.4, 82.5)
- removed the REF** at (63.5, 25.4)
- added REF**: CUTOUT_MX_1.00u, Caon_Footprint:Cutout_MX_1.00u, F.Cu at (158.8, 25.4)
- added REF**: CUTOUT_MX_1.00u, Caon_Footprint:Cutout_MX_1.00u, F.Cu at (54.0, 44.5)
- added REF**: CUTOUT_MX_1.00u, Caon_Footprint:Cutout_MX_1.00u, F.Cu at (44.5, 101.6)
- added REF**: CUTOUT_MX_1.00u, Caon_Footprint:Cutout_MX_1.00u, F.Cu at (68.3, 82.5)
- added REF**: CUTOUT_MX_1.00u, Caon_Footprint:Cutout_MX_1.00u, F.Cu at (92.1, 44.5)
- added REF**: CUTOUT_MX_1.00u, Caon_Footprint:Cutout_MX_1.00u, F.Cu at (25.4, 25.4)
- added REF**: CUTOUT_MX_1.00u, Caon_Footprint:Cutout_MX_1.00u, F.Cu at (154.0, 63.5)
- added REF**: CUTOUT_MX_1.00u, Caon_Footprint:Cutout_MX_1.00u, F.Cu at (149.2, 101.6)
- added REF**: CUTOUT_MX_1.00u, Caon_Footprint:Cutout_MX_1.00u, F.Cu at (82.5, 25.4)
- added REF**: CUTOUT_MX_1.00u, Caon_Footprint:Cutout_MX_1.00u, F.Cu at (230.2, 63.5)
- added REF**: CUTOUT_MX_1.00u, Caon_Footprint:Cutout_MX_1.00u, F.Cu at (130.2, 44.5)
- added REF**: CUTOUT_MX_1.00u, Caon_Footprint:Cutout_MX_1.00u, F.Cu at (139.7, 25.4)
- added REF**: CUTOUT_MX_1.00u, Caon_Footprint:Cutout_MX_1.00u, F.Cu at (120.7, 25.4)
- added REF**: CUTOUT_MX_1.00u, Caon_Footprint:Cutout_MX_1.00u, F.Cu at (125.4, 82.5)
- added REF**: CUTOUT_MX_1.00u, Caon_Footprint:Cutout_MX_1.00u, F.Cu at (244.5, 44.5)
- added REF**: CUTOUT_MX_1.00u, Caon_Footprint:Cutout_MX_1.00u, F.Cu at (234.9, 101.6)
- added REF**: CUTOUT_MX_1.00u, Caon_Footprint:Cutout_MX_1.00u, F.Cu at (49.2, 82.5)
- added REF**: CUTOUT_MX_1.00u, Caon_Footprint:Cutout_MX_1.00u, F.Cu at (196.8, 25.4)
- added REF**: CUTOUT_MX_1.00u, Caon_Footprint:Cutout_MX_1.00u, F.Cu at (254.0, 101.6)
- added REF**: CUTOUT_MX_1.00u, Caon_Footprint:Cutout_MX_1.00u, F.Cu at (144.5, 82.5)
- added REF**: CUTOUT_MX_1.00u, Caon_Footprint:Cutout_MX_1.00u, F.Cu at (201.6, 82.5)
- added REF**: CUTOUT_MX_1.00u, Caon_Footprint:Cutout_MX_1.00u, F.Cu at (101.6, 25.4)
- added REF**: CUTOUT_MX_1.00u, Caon_Footprint:Cutout_MX_1.00u, F.Cu at (63.5, 25.4)
- added REF**: CUTOUT_MX_1.00u, Caon_Footprint:Cutout_MX_1.00u, F.Cu at (273.1, 25.4)
- added REF**: CUTOUT_MX_1.00u, Caon_Footprint:Cutout_MX_1.00u, F.Cu at (177.8, 25.4)
- added REF**: CUTOUT_MX_1.00u, Caon_Footprint:Cutout_MX_1.00u, F.Cu at (187.3, 44.5)
- added REF**: CUTOUT_MX_1.00u, Caon_Footprint:Cutout_MX_1.00u, F.Cu at (206.4, 44.5)
- added REF**: CUTOUT_MX_1.00u, Caon_Footprint:Cutout_MX_1.00u, F.Cu at (311.1, 101.6)
- added REF**: CUTOUT_MX_1.00u, Caon_Footprint:Cutout_MX_1.00u, F.Cu at (225.4, 44.5)
- added REF**: CUTOUT_MX_1.00u, Caon_Footprint:Cutout_MX_1.00u, F.Cu at (149.2, 44.5)
- added REF**: CUTOUT_MX_1.00u, Caon_Footprint:Cutout_MX_1.00u, F.Cu at (192.1, 63.5)
- added REF**: CUTOUT_MX_1.00u, Caon_Footprint:Cutout_MX_1.00u, F.Cu at (220.7, 82.5)
- added REF**: CUTOUT_MX_1.00u, Caon_Footprint:Cutout_MX_1.00u, F.Cu at (168.3, 44.5)
- added REF**: CUTOUT_MX_1.00u, Caon_Footprint:Cutout_MX_1.00u, F.Cu at (215.9, 101.6)
- added REF**: CUTOUT_MX_1.00u, Caon_Footprint:Cutout_MX_1.00u, F.Cu at (130.2, 101.6)
- added REF**: CUTOUT_MX_1.00u, Caon_Footprint:Cutout_MX_1.00u, F.Cu at (58.7, 63.5)
- added REF**: CUTOUT_MX_1.00u, Caon_Footprint:Cutout_MX_1.00u, F.Cu at (111.1, 44.5)
- added REF**: CUTOUT_MX_1.00u, Caon_Footprint:Cutout_MX_1.00u, F.Cu at (87.3, 82.5)
- added REF**: CUTOUT_MX_1.00u, Caon_Footprint:Cutout_MX_1.00u, F.Cu at (106.4, 82.5)
- added REF**: CUTOUT_MX_1.00u, Caon_Footprint:Cutout_MX_1.00u, F.Cu at (292.1, 25.4)
- added REF**: CUTOUT_MX_1.00u, Caon_Footprint:Cutout_MX_1.00u, F.Cu at (163.5, 82.5)
- added REF**: CUTOUT_MX_1.00u, Caon_Footprint:Cutout_MX_1.00u, F.Cu at (249.2, 63.5)
- added REF**: CUTOUT_MX_1.00u, Caon_Footprint:Cutout_MX_1.00u, F.Cu at (239.7, 82.5)
- added REF**: CUTOUT_MX_1.00u, Caon_Footprint:Cutout_MX_1.00u, F.Cu at (25.4, 101.6)
- added REF**: CUTOUT_MX_1.00u, Caon_Footprint:Cutout_MX_1.00u, F.Cu at (44.5, 25.4)
- added REF**: CUTOUT_MX_1.00u, Caon_Footprint:Cutout_MX_1.00u, F.Cu at (63.5, 101.6)
- added REF**: CUTOUT_MX_1.00u, Caon_Footprint:Cutout_MX_1.00u, F.Cu at (292.1, 82.5)
- added REF**: CUTOUT_MX_1.00u, Caon_Footprint:Cutout_MX_1.00u, F.Cu at (77.8, 63.5)
- added REF**: CUTOUT_MX_1.00u, Caon_Footprint:Cutout_MX_1.00u, F.Cu at (134.9, 63.5)
- added REF**: CUTOUT_MX_1.00u, Caon_Footprint:Cutout_MX_1.00u, F.Cu at (292.1, 101.6)
- added REF**: CUTOUT_MX_1.00u, Caon_Footprint:Cutout_MX_1.00u, F.Cu at (168.3, 101.6)
- added REF**: CUTOUT_MX_1.00u, Caon_Footprint:Cutout_MX_1.00u, F.Cu at (82.5, 101.6)
- added REF**: CUTOUT_MX_1.00u, Caon_Footprint:Cutout_MX_1.00u, F.Cu at (234.9, 25.4)
- added REF**: CUTOUT_MX_1.00u, Caon_Footprint:Cutout_MX_1.00u, F.Cu at (173.0, 63.5)
- added REF**: CUTOUT_MX_1.00u, Caon_Footprint:Cutout_MX_1.00u, F.Cu at (96.8, 63.5)
- added REF**: CUTOUT_MX_1.00u, Caon_Footprint:Cutout_MX_1.00u, F.Cu at (215.9, 25.4)
- added REF**: CUTOUT_MX_1.00u, Caon_Footprint:Cutout_MX_1.00u, F.Cu at (268.3, 63.5)
- added REF**: CUTOUT_MX_1.00u, Caon_Footprint:Cutout_MX_1.00u, F.Cu at (211.1, 63.5)
- added REF**: CUTOUT_MX_1.00u, Caon_Footprint:Cutout_MX_1.00u, F.Cu at (254.0, 25.4)
- added REF**: CUTOUT_MX_1.00u, Caon_Footprint:Cutout_MX_1.00u, F.Cu at (263.5, 44.5)
- added REF**: CUTOUT_MX_1.00u, Caon_Footprint:Cutout_MX_1.00u, F.Cu at (73.0, 44.5)
- added REF**: CUTOUT_MX_1.00u, Caon_Footprint:Cutout_MX_1.00u, F.Cu at (115.9, 63.5)
- added REF**: CUTOUT_MX_1.00u, Caon_Footprint:Cutout_MX_1.00u, F.Cu at (273.1, 101.6)
- added REF**: CUTOUT_MX_1.00u, Caon_Footprint:Cutout_MX_1.00u, F.Cu at (182.6, 82.5)

Commit message: Plate Update
Parts:
- removed the REF** at (27.8, 82.5)
- removed the REF** at (32.5, 63.5)
- removed the REF** at (289.7, 63.5)
- removed the REF** at (287.3, 44.5)
- removed the REF** at (265.9, 82.5)
- removed the REF** at (30.2, 44.5)
- removed the REF** at (106.4, 101.6)
- removed the REF** at (192.1, 101.6)
- added REF**: MountingHole_2.2mm_M2, MountingHole:MountingHole_2.2mm_M2, F.Cu at (201.6, 63.5)
- added REF**: CUTOUT_MX_1.25u, Caon_Footprint:Cutout_MX_1.25u, F.Cu at (289.7, 63.5)
- added REF**: CUTOUT_MX_1.50u, Caon_Footprint:Cutout_MX_1.50u, F.Cu at (106.4, 101.6)
- added REF**: CUTOUT_MX_1.50u, Caon_Footprint:Cutout_MX_1.50u, F.Cu at (30.2, 44.5)
- added REF**: CUTOUT_MX_1.75u, Caon_Footprint:Cutout_MX_1.75u, F.Cu at (265.9, 82.5)
- added REF**: CUTOUT_MX_1.75u, Caon_Footprint:Cutout_MX_1.75u, F.Cu at (32.5, 63.5)
- added REF**: CUTOUT_MX_1.50u, Caon_Footprint:Cutout_MX_1.50u, F.Cu at (287.3, 44.5)
- added REF**: CUTOUT_MX_1.25u, Caon_Footprint:Cutout_MX_1.25u, F.Cu at (27.8, 82.5)
- added REF**: CUTOUT_MX_1.50u, Caon_Footprint:Cutout_MX_1.50u, F.Cu at (192.1, 101.6)
- moved REF** 38.1 mm to (125.4, 63.5)
- moved REF** 1.59 mm to (279.4, 63.5)

Commit message: Final
Parts:
- removed the REF** at (311.1, 20.6)
- removed the REF** at (201.6, 63.5)
- removed the REF** at (34.9, 20.6)
- removed the REF** at (301.6, 106.4)
- removed the REF** at (46.0, 63.5)
- removed the REF** at (225.4, 20.6)
- removed the REF** at (125.4, 63.5)
- removed the REF** at (34.9, 106.4)
- removed the REF** at (111.1, 20.6)
- removed the REF** at (279.4, 63.5)
- removed the REF** at (94.5, 106.4)
- removed the REF** at (204.0, 106.4)
Other:
- outline, holes or cut-outs redrawn

Commit message: Back to drawing board
Parts:
- removed the REF** at (158.8, 25.4)
- removed the REF** at (92.1, 44.5)
- removed the REF** at (154.0, 63.5)
- removed the REF** at (82.5, 25.4)
- removed the REF** at (230.2, 63.5)
- removed the REF** at (130.2, 44.5)
- removed the REF** at (139.7, 25.4)
- removed the REF** at (120.7, 25.4)
- removed the REF** at (125.4, 82.5)
- removed the REF** at (149.2, 101.6)
- removed the REF** at (244.5, 44.5)
- removed the REF** at (234.9, 101.6)
- removed the REF** at (196.8, 25.4)
- removed the REF** at (254.0, 101.6)
- removed the REF** at (144.5, 82.5)
- removed the REF** at (201.6, 82.5)
- removed the REF** at (101.6, 25.4)
- removed the REF** at (63.5, 25.4)
- removed the REF** at (273.1, 25.4)
- removed the REF** at (177.8, 25.4)
- removed the REF** at (49.2, 82.5)
- removed the REF** at (289.7, 63.5)
- removed the REF** at (206.4, 44.5)
- removed the REF** at (311.1, 101.6)
- removed the REF** at (225.4, 44.5)
- removed the REF** at (149.2, 44.5)
- removed the REF** at (192.1, 63.5)
- removed the REF** at (220.7, 82.5)
- removed the REF** at (106.4, 101.6)
- removed the REF** at (168.3, 44.5)
- removed the REF** at (215.9, 101.6)
- removed the REF** at (187.3, 44.5)
- removed the REF** at (130.2, 101.6)
- removed the REF** at (58.7, 63.5)
- removed the REF** at (111.1, 44.5)
- removed the REF** at (87.3, 82.5)
- removed the REF** at (106.4, 82.5)
- removed the REF** at (292.1, 25.4)
- removed the REF** at (163.5, 82.5)
- removed the REF** at (249.2, 63.5)
- removed the REF** at (30.2, 44.5)
- removed the REF** at (239.7, 82.5)
- removed the REF** at (292.1, 101.6)
- removed the REF** at (25.4, 101.6)
- removed the REF** at (265.9, 82.5)
- removed the REF** at (44.5, 25.4)
- removed the REF** at (63.5, 101.6)
- removed the REF** at (292.1, 82.5)
- removed the REF** at (77.8, 63.5)
- removed the REF** at (32.5, 63.5)
- removed the REF** at (134.9, 63.5)
- removed the REF** at (168.3, 101.6)
- removed the REF** at (82.5, 101.6)
- removed the REF** at (182.6, 82.5)
- removed the REF** at (234.9, 25.4)
- removed the REF** at (287.3, 44.5)
- removed the REF** at (173.0, 63.5)
- removed the REF** at (96.8, 63.5)
- removed the REF** at (215.9, 25.4)
- removed the REF** at (268.3, 63.5)
- removed the REF** at (211.1, 63.5)
- removed the REF** at (254.0, 25.4)
- removed the REF** at (263.5, 44.5)
- removed the REF** at (54.0, 44.5)
- removed the REF** at (73.0, 44.5)
- removed the REF** at (27.8, 82.5)
- removed the REF** at (115.9, 63.5)
- removed the REF** at (192.1, 101.6)
- removed the REF** at (273.1, 101.6)
- removed the REF** at (44.5, 101.6)
- removed the REF** at (68.3, 82.5)

Commit message: New Update
Parts:
- added REF**: CUTOUT_MX_1.00u, Caon_Footprint:Cutout_MX_1.00u, F.Cu at (201.6, 82.5)
- added REF**: CUTOUT_MX_1.00u, Caon_Footprint:Cutout_MX_1.00u, F.Cu at (120.7, 25.4)
- added REF**: CUTOUT_MX_1.00u, Caon_Footprint:Cutout_MX_1.00u, F.Cu at (163.5, 82.5)
- added REF**: CUTOUT_MX_1.00u, Caon_Footprint:Cutout_MX_1.00u, F.Cu at (82.5, 101.6)
- added REF**: CUTOUT_MX_1.00u, Caon_Footprint:Cutout_MX_1.00u, F.Cu at (130.2, 101.6)
- added REF**: CUTOUT_MX_1.00u, Caon_Footprint:Cutout_MX_1.00u, F.Cu at (273.1, 101.6)
- added REF**: CUTOUT_MX_1.00u, Caon_Footprint:Cutout_MX_1.00u, F.Cu at (215.9, 25.4)
- added REF**: CUTOUT_MX_1.00u, Caon_Footprint:Cutout_MX_1.00u, F.Cu at (77.8, 63.5)
- added REF**: CUTOUT_MX_1.00u, Caon_Footprint:Cutout_MX_1.00u, F.Cu at (125.4, 82.5)
- added REF**: CUTOUT_MX_1.00u, Caon_Footprint:Cutout_MX_1.00u, F.Cu at (106.4, 82.5)
- added REF**: CUTOUT_MX_1.50u, Caon_Footprint:Cutout_MX_1.50u, F.Cu at (106.4, 101.6)
- added REF**: CUTOUT_MX_1.00u, Caon_Footprint:Cutout_MX_1.00u, F.Cu at (144.5, 82.5)
- added REF**: CUTOUT_MX_1.00u, Caon_Footprint:Cutout_MX_1.00u, F.Cu at (149.2, 44.5)
- added REF**: CUTOUT_MX_1.00u, Caon_Footprint:Cutout_MX_1.00u, F.Cu at (154.0, 63.5)
- added REF**: CUTOUT_MX_1.00u, Caon_Footprint:Cutout_MX_1.00u, F.Cu at (292.1, 101.6)
- added REF**: CUTOUT_MX_1.00u, Caon_Footprint:Cutout_MX_1.00u, F.Cu at (63.5, 25.4)
- added REF**: CUTOUT_MX_1.00u, Caon_Footprint:Cutout_MX_1.00u, F.Cu at (192.1, 63.5)
- added REF**: CUTOUT_MX_1.00u, Caon_Footprint:Cutout_MX_1.00u, F.Cu at (139.7, 25.4)
- added REF**: CUTOUT_MX_1.00u, Caon_Footprint:Cutout_MX_1.00u, F.Cu at (177.8, 25.4)
- added REF**: CUTOUT_MX_1.00u, Caon_Footprint:Cutout_MX_1.00u, F.Cu at (254.0, 101.6)
- added REF**: CUTOUT_MX_1.00u, Caon_Footprint:Cutout_MX_1.00u, F.Cu at (134.9, 63.5)
- added REF**: CUTOUT_MX_1.25u, Caon_Footprint:Cutout_MX_1.25u, F.Cu at (27.8, 82.5)
- added REF**: CUTOUT_MX_1.00u, Caon_Footprint:Cutout_MX_1.00u, F.Cu at (225.4, 44.5)
- added REF**: CUTOUT_MX_1.00u, Caon_Footprint:Cutout_MX_1.00u, F.Cu at (49.2, 82.5)
- added REF**: CUTOUT_MX_1.00u, Caon_Footprint:Cutout_MX_1.00u, F.Cu at (73.0, 44.5)
- added REF**: CUTOUT_MX_1.75u, Caon_Footprint:Cutout_MX_1.75u, F.Cu at (265.9, 82.5)
- added REF**: CUTOUT_MX_1.00u, Caon_Footprint:Cutout_MX_1.00u, F.Cu at (215.9, 101.6)
- added REF**: CUTOUT_MX_1.00u, Caon_Footprint:Cutout_MX_1.00u, F.Cu at (101.6, 25.4)
- added REF**: CUTOUT_MX_1.00u, Caon_Footprint:Cutout_MX_1.00u, F.Cu at (168.3, 101.6)
- added REF**: CUTOUT_MX_1.00u, Caon_Footprint:Cutout_MX_1.00u, F.Cu at (130.2, 44.5)
- added REF**: CUTOUT_MX_1.00u, Caon_Footprint:Cutout_MX_1.00u, F.Cu at (149.2, 101.6)
- added REF**: CUTOUT_MX_1.00u, Caon_Footprint:Cutout_MX_1.00u, F.Cu at (268.3, 63.5)
- added REF**: CUTOUT_MX_1.00u, Caon_Footprint:Cutout_MX_1.00u, F.Cu at (273.1, 25.4)
- added REF**: CUTOUT_MX_1.00u, Caon_Footprint:Cutout_MX_1.00u, F.Cu at (196.8, 25.4)
- added REF**: CUTOUT_MX_1.00u, Caon_Footprint:Cutout_MX_1.00u, F.Cu at (158.8, 25.4)
- added REF**: CUTOUT_MX_1.00u, Caon_Footprint:Cutout_MX_1.00u, F.Cu at (220.7, 82.5)
- added REF**: CUTOUT_MX_1.00u, Caon_Footprint:Cutout_MX_1.00u, F.Cu at (239.7, 82.5)
- added REF**: CUTOUT_MX_1.00u, Caon_Footprint:Cutout_MX_1.00u, F.Cu at (230.2, 63.5)
- added REF**: CUTOUT_MX_1.00u, Caon_Footprint:Cutout_MX_1.00u, F.Cu at (96.8, 63.5)
- added REF**: CUTOUT_MX_1.00u, Caon_Footprint:Cutout_MX_1.00u, F.Cu at (211.1, 63.5)
- added REF**: CUTOUT_MX_1.00u, Caon_Footprint:Cutout_MX_1.00u, F.Cu at (54.0, 44.5)
- added REF**: CUTOUT_MX_1.00u, Caon_Footprint:Cutout_MX_1.00u, F.Cu at (182.6, 82.5)
- added REF**: CUTOUT_MX_1.00u, Caon_Footprint:Cutout_MX_1.00u, F.Cu at (115.9, 63.5)
- added REF**: CUTOUT_MX_1.00u, Caon_Footprint:Cutout_MX_1.00u, F.Cu at (111.1, 44.5)
- added REF**: CUTOUT_MX_1.00u, Caon_Footprint:Cutout_MX_1.00u, F.Cu at (234.9, 25.4)
- added REF**: CUTOUT_MX_1.00u, Caon_Footprint:Cutout_MX_1.00u, F.Cu at (44.5, 101.6)
- added REF**: CUTOUT_MX_1.00u, Caon_Footprint:Cutout_MX_1.00u, F.Cu at (173.0, 63.5)
- added REF**: CUTOUT_MX_1.00u, Caon_Footprint:Cutout_MX_1.00u, F.Cu at (68.3, 82.5)
- added REF**: CUTOUT_MX_1.00u, Caon_Footprint:Cutout_MX_1.00u, F.Cu at (92.1, 44.5)
- added REF**: CUTOUT_MX_1.00u, Caon_Footprint:Cutout_MX_1.00u, F.Cu at (63.5, 101.6)
- added REF**: CUTOUT_MX_1.00u, Caon_Footprint:Cutout_MX_1.00u, F.Cu at (58.7, 63.5)
- added REF**: CUTOUT_MX_1.00u, Caon_Footprint:Cutout_MX_1.00u, F.Cu at (206.4, 44.5)
- added REF**: CUTOUT_MX_1.00u, Caon_Footprint:Cutout_MX_1.00u, F.Cu at (249.2, 63.5)
- added REF**: CUTOUT_MX_1.00u, Caon_Footprint:Cutout_MX_1.00u, F.Cu at (292.1, 82.5)
- added REF**: CUTOUT_MX_1.00u, Caon_Footprint:Cutout_MX_1.00u, F.Cu at (244.5, 44.5)
- added REF**: CUTOUT_MX_1.75u, Caon_Footprint:Cutout_MX_1.75u, F.Cu at (32.5, 63.5)
- added REF**: CUTOUT_MX_1.00u, Caon_Footprint:Cutout_MX_1.00u, F.Cu at (25.4, 101.6)
- added REF**: CUTOUT_MX_1.00u, Caon_Footprint:Cutout_MX_1.00u, F.Cu at (82.5, 25.4)
- added REF**: CUTOUT_MX_1.00u, Caon_Footprint:Cutout_MX_1.00u, F.Cu at (44.5, 25.4)
- added REF**: CUTOUT_MX_1.00u, Caon_Footprint:Cutout_MX_1.00u, F.Cu at (87.3, 82.5)
- added REF**: CUTOUT_MX_1.50u, Caon_Footprint:Cutout_MX_1.50u, F.Cu at (287.3, 44.5)
- added REF**: CUTOUT_MX_1.00u, Caon_Footprint:Cutout_MX_1.00u, F.Cu at (168.3, 44.5)
- added REF**: CUTOUT_MX_1.00u, Caon_Footprint:Cutout_MX_1.00u, F.Cu at (254.0, 25.4)
- added REF**: CUTOUT_MX_1.00u, Caon_Footprint:Cutout_MX_1.00u, F.Cu at (311.1, 101.6)
- added REF**: CUTOUT_MX_1.00u, Caon_Footprint:Cutout_MX_1.00u, F.Cu at (187.3, 44.5)
- added REF**: CUTOUT_MX_1.00u, Caon_Footprint:Cutout_MX_1.00u, F.Cu at (263.5, 44.5)
- added REF**: CUTOUT_MX_1.50u, Caon_Footprint:Cutout_MX_1.50u, F.Cu at (192.1, 101.6)
- added REF**: CUTOUT_MX_1.00u, Caon_Footprint:Cutout_MX_1.00u, F.Cu at (292.1, 25.4)
- added REF**: CUTOUT_MX_1.00u, Caon_Footprint:Cutout_MX_1.00u, F.Cu at (234.9, 101.6)
- added REF**: CUTOUT_MX_1.25u, Caon_Footprint:Cutout_MX_1.25u, F.Cu at (289.7, 63.5)
- added REF**: CUTOUT_MX_1.50u, Caon_Footprint:Cutout_MX_1.50u, F.Cu at (30.2, 44.5)

Commit message: Dxf plate Desing Done
Other:
- board text removed: "REF**"
